File: MPR121 Template/MPR121 Template.sch (KiCad schematic (older format))
At the start: 7 parts

Commit message: Template added
Parts:
- added J1: Conn_01x03_Male, CCHS:Touch_Slider_Shielded, symbol Connector:Conn_01x03_Male
- C1, C2: renamed from C?; footprint (none) -> Capacitors_SMD:C_0805_HandSoldering
- R1, R2, R3: renamed from R?; footprint (none) -> Resistors_SMD:R_0805_HandSoldering
- U1: renamed from U?; footprint (none) -> CCHS:SAO_Header_6-Pin
- U2: renamed from U?; footprint (none) -> Housings_DFN_QFN:SiliconLabs_QFN-20-1EP_3x3mm_Pitch0.5mm
Connections:
- net GND: now also J1.3 (Pin_3)
Changed lines of the file:
@@
 $EndDescr
 $Comp
-L CCHS:MPR121 U?
+L CCHS:MPR121 U2
 U 1 1 5F840BA0
 P 5600 3350
-F 0 "U?" H 5600 4115 50  0000 C CNN
+F 0 "U2" H 5600 4115 50  0000 C CNN
 F 1 "MPR121" H 5600 4024 50  0000 C CNN
-F 2 "" H 5500 2850 50  0001 C CNN
+F 2 "Housings_DFN_QFN:SiliconLabs_QFN-20-1EP_3x3mm_Pitch0.5mm" H 5500 2850 50  0001 C CNN
 F 3 "" H 5500 2850 50  0001 C CNN
 	1    5600 3350
@@
 $EndComp
 $Comp
-L CCHS:SAO U?
+L CCHS:SAO U1
 U 1 1 5F8415A9
 P 2550 3350
-F 0 "U?" H 2550 3715 50  0000 C CNN
+F 0 "U1" H 2550 3715 50  0000 C CNN
 F 1 "SAO" H 2550 3624 50  0000 C CNN
-F 2 "" H 2550 3150 50  0001 C CNN
+F 2 "CCHS:SAO_Header_6-Pin" H 2550 3150 50  0001 C CNN
 F 3 "" H 2550 3150 50  0001 C CNN
 	1    2550 3350
@@
 	2200 3250 2000 3250
 $Comp
-L power:GND #PWR?
+L power:GND #PWR0101
 U 1 1 5F844599
 P 2000 4050
-F 0 "#PWR?" H 2000 3800 50  0001 C CNN
+F 0 "#PWR0101" H 2000 3800 50  0001 C CNN
 F 1 "GND" H 2005 3877 50  0000 C CNN
 F 2 "" H 2000 4050 50  0001 C CNN
@@
 	4100 2950 4100 3450
 $Comp
-L power:GND #PWR?
+L power:GND #PWR0102
 U 1 1 5F846111
 P 4100 4050
-F 0 "#PWR?" H 4100 3800 50  0001 C CNN
+F 0 "#PWR0102" H 4100 3800 50  0001 C CNN
 F 1 "GND" H 4105 3877 50  0000 C CNN
 F 2 "" H 4100 4050 50  0001 C CNN
@@
 	5100 2650 5100 2850
 $Comp
-L Device:C C?
+L Device:C C1
 U 1 1 5F846AE4
 P 4600 2800
-F 0 "C?" H 4715 2846 50  0000 L CNN
+F 0 "C1" H 4715 2846 50  0000 L CNN
 F 1 "0.1uF" H 4715 2755 50  0000 L CNN
-F 2 "" H 4638 2650 50  0001 C CNN
+F 2 "Capacitors_SMD:C_0805_HandSoldering" H 4638 2650 50  0001 C CNN
 F 3 "~" H 4600 2800 50  0001 C CNN
 	1    4600 2800
@@
 $EndComp
 $Comp
-L Device:C C?
+L Device:C C2
 U 1 1 5F84A0C4
 P 4350 3650
-F 0 "C?" H 4465 3696 50  0000 L CNN
+F 0 "C2" H 4465 3696 50  0000 L CNN
 F 1 "0.1uF" H 4465 3605 50  0000 L CNN
-F 2 "" H 4388 3500 50  0001 C CNN
+F 2 "Capacitors_SMD:C_0805_HandSoldering" H 4388 3500 50  0001 C CNN
 F 3 "~" H 4350 3650 50  0001 C CNN
 	1    4350 3650
@@
 	4350 3050 4350 3500
 $Comp
-L power:GND #PWR?
+L power:GND #PWR0103
 U 1 1 5F84ADE1
 P 4350 4050
-F 0 "#PWR?" H 4350 3800 50  0001 C CNN
+F 0 "#PWR0103" H 4350 3800 50  0001 C CNN
 F 1 "GND" H 4355 3877 50  0000 C CNN
 F 2 "" H 4350 4050 50  0001 C CNN
@@
 	4100 3450 4100 4050
 $Comp
-L power:GND #PWR?
+L power:GND #PWR0104
 U 1 1 5F84BAE5
 P 4800 4050
-F 0 "#PWR?" H 4800 3800 50  0001 C CNN
+F 0 "#PWR0104" H 4800 3800 50  0001 C CNN
 F 1 "GND" H 4805 3877 50  0000 C CNN
 F 2 "" H 4800 4050 50  0001 C CNN
@@
 	2900 3250 2900 2650
 $Comp
-L Device:R R?
+L Device:R R1
 U 1 1 5F853B52
 P 3150 3000
-F 0 "R?" H 3220 3046 50  0000 L CNN
+F 0 "R1" H 3220 3046 50  0000 L CNN
 F 1 "R" H 3220 2955 50  0000 L CNN
-F 2 "" V 3080 3000 50  0001 C CNN
+F 2 "Resistors_SMD:R_0805_HandSoldering" V 3080 3000 50  0001 C CNN
 F 3 "~" H 3150 3000 50  0001 C CNN
 	1    3150 3000
@@
 $EndComp
 $Comp
-L Device:R R?
+L Device:R R2
 U 1 1 5F853D5F
 P 3400 3000
-F 0 "R?" H 3470 3046 50  0000 L CNN
+F 0 "R2" H 3470 3046 50  0000 L CNN
 F 1 "R" H 3470 2955 50  0000 L CNN
-F 2 "" V 3330 3000 50  0001 C CNN
+F 2 "Resistors_SMD:R_0805_HandSoldering" V 3330 3000 50  0001 C CNN
 F 3 "~" H 3400 3000 50  0001 C CNN
 	1    3400 3000
@@
 $EndComp
 $Comp
-L Device:R R?
+L Device:R R3
 U 1 1 5F853F89
 P 3650 3000
-F 0 "R?" H 3720 3046 50  0000 L CNN
+F 0 "R3" H 3720 3046 50  0000 L CNN
 F 1 "R" H 3720 2955 50  0000 L CNN
-F 2 "" V 3580 3000 50  0001 C CNN
+F 2 "Resistors_SMD:R_0805_HandSoldering" V 3580 3000 50  0001 C CNN
 F 3 "~" H 3650 3000 50  0001 C CNN
 	1    3650 3000
@@
 Wire Wire Line
 	4100 2950 4600 2950
+$Comp
+L Connector:Conn_01x03_Male J1
+U 1 1 5F84DB13
+P 7800 3100
+F 0 "J1" H 7908 3381 50  0000 C CNN
+F 1 "Conn_01x03_Male" H 7908 3290 50  0000 C CNN
+F 2 "CCHS:Touch_Slider_Shielded" H 7800 3100 50  0001 C CNN
+F 3 "~" H 7800 3100 50  0001 C CNN
+	1    7800 3100
+	1    0    0    -1
+$EndComp
+$Comp
+L power:GND #PWR0105
+U 1 1 5F84E5C5
+P 8000 3200
+F 0 "#PWR0105" H 8000 2950 50  0001 C CNN
+F 1 "GND" H 8005 3027 50  0000 C CNN
+F 2 "" H 8000 3200 50  0001 C CNN
+F 3 "" H 8000 3200 50  0001 C CNN
+	1    8000 3200
+	1    0    0    -1
+$EndComp
 $EndSCHEMATC
